File: ASM2464PD-test.kicad_sch (KiCad schematic)
At the start: 41 parts, among them J1 USB_C_Receptacle, J2 Bus_M.2_Socket_M

Commit message: Added SPI flash, probably some more stuff, and made pcb 4-layer
Parts:
- added C17: 1u, Capacitor_SMD:C_0201_0603Metric, symbol Device:C_Small
- added C18: 0.1u, Capacitor_SMD:C_0201_0603Metric, symbol Device:C_Small
- added R15, R17, R18: 4.7k, Resistor_SMD:R_0201_0603Metric, symbol Device:R_Small
- added R16: 10k, Resistor_SMD:R_0201_0603Metric, symbol Device:R_Small
- added R19, R20, R21: 0Ω, Resistor_SMD:R_0201_0603Metric, symbol Device:R_Small
- added U2: SPI_SOIC-8, Package_SO:SOIC-8_5.23x5.23mm_P1.27mm, symbol A_my_stuff:SPI_flash
- added U3: SPI_DFN-8, Package_DFN_QFN:DFN-8-1EP_3x2mm_P0.5mm_EP1.3x1.5mm, symbol A_my_stuff:SPI_flash
- R13, R14: value 2M -> 0Ω
Connections:
- net CC1: now also R13.2; no longer J1.A5 (CC1)
- net CC2: now also R14.2; no longer J1.B5 (CC2)
- net GND: now also C17.2, C18.2, R16.2, U2.4 (GND), U3.4 (GND); no longer R13.2, R14.2
- net PERST#: now also U1.G21 (PERST0#), R19.1; no longer J2.50 (~{PERST})
- net SBU1_C: no longer R13.1
- net SBU2_C: no longer R14.1
- net +5V_VBUS: now reaches J1.A4 (VBUS), J1.A9 (VBUS), J1.B4 (VBUS), J1.B9 (VBUS)
- net +5V_VBUS: now also R15.1
- net at J2.52 (~{CLKREQ}): now also R20.2
- net at J2.54 (~{PEWAKE}): now also R21.2
- net SPI_CS#: now reaches U1.A2 (SPI_CS#)
- net SPI_CS#: now also U2.1 (~{CS}), U3.1 (~{CS})
- net SPI_DO: now reaches U1.A3 (SPI_DO)
- net SPI_DO: now also U2.5 (MOSI), U3.5 (MOSI)
- net SPI_DI: now reaches U1.A4 (SPI_DI)
- net SPI_DI: now also U2.2 (MISO), U3.2 (MISO)
- net SPI_CLK: now reaches U1.A5 (SPI_CLK)
- net SPI_CLK: now also U2.6 (SCK), U3.6 (SCK)
- net VBUS: now reaches U1.G1 (VBUS)
- net VBUS: now also C17.1, R15.2, R16.1
- net 3.3V renamed +3.3V
- net +3.3V: now also C18.1, R17.2, R18.2, U2.8 (VCC), U3.8 (VCC)
- net 3.3VA renamed +3.3VA
- new net: J2.50 (~{PERST}), R19.2
- new net CC1_C: J1.A5 (CC1), R13.1
- new net CC2_C: J1.B5 (CC2), R14.1
- new net SPI_HOLD#: R17.1, U2.7 (~{HOLD}), U3.7 (~{HOLD})
- new net SPI_WP#: R18.1, U2.3 (~{WP}), U3.3 (~{WP})
Other:
- note added: "todo idk weird"
- moved on the sheet: C1, C2, C3, C4, C5, C6, C7, C8, J2
